File: 40Hz Light Sound.kicad_sch (KiCad schematic)
At the start: 8 parts, among them J1 11.1VDC, J2 DC2DC, J3 Audio_Amp, J4 LED_Conn, J5 AudioJack3_Ground, Q1 IRLZ44N, SW1 SW_SPDT, U1 ESP32-C3_SUPERMINI_TH

Commit message: Submit v0.1 to order
Parts:
- J1, J4: footprint Connector_AMASS:AMASS_XT30PW-M_1x02_P2.50mm_Horizontal -> Connector_JST:JST_GH_SM02B-GHS-TB_1x02-1MP_P1.25mm_Horizontal
- Q1: value IRLZ44N -> IRLML6344; footprint IRLZ44N:TO254P1054X469X1930-3 -> IRLML6344TRPBF:SOT95P240X112-3N
Other:
- moved on the sheet: Q1
Changed lines of the file:
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@@
 	(global_label "LED_GND"
 		(shape input)
-		(at 203.2 76.2 180)
+		(at 194.31 76.2 180)
 		(fields_autoplaced yes)
 		(effects
@@
 		)
 		(property "Intersheetrefs" "${INTERSHEET_REFS}"
-			(at 191.9296 76.2 0)
+			(at 183.0396 76.2 0)
 			(effects
 				(font
@@
 	(global_label "GND"
 		(shape passive)
-		(at 203.2 86.36 0)
+		(at 194.31 86.36 0)
 		(fields_autoplaced yes)
 		(effects
@@
 		)
 		(property "Intersheetrefs" "${INTERSHEET_REFS}"
-			(at 208.9444 86.36 0)
+			(at 200.0544 86.36 0)
 			(effects
 				(font
@@
 	(global_label "LEDcontrol"
 		(shape input)
-		(at 198.12 83.82 180)
+		(at 189.23 83.82 180)
 		(fields_autoplaced yes)
 		(effects
@@
 		)
 		(property "Intersheetrefs" "${INTERSHEET_REFS}"
-			(at 184.975 83.82 0)
+			(at 176.085 83.82 0)
 			(effects
 				(font
@@
 	(symbol
 		(lib_id "IRLZ44N:IRLZ44N")
-		(at 200.66 81.28 0)
+		(at 191.77 81.28 0)
 		(unit 1)
 		(exclude_from_sim no)
@@
 		(fields_autoplaced yes)
 		(property "Reference" "Q1"
-			(at 207.01 80.0099 0)
-			(effects
-				(font
-					(size 1.27 1.27)
-				)
-				(justify left)
-			)
-		)
-		(property "Value" "IRLZ44N"
-			(at 207.01 82.5499 0)
-			(effects
-				(font
-					(size 1.27 1.27)
-				)
-				(justify left)
-			)
-		)
-		(property "Footprint" "IRLZ44N:TO254P1054X469X1930-3"
-			(at 200.66 81.28 0)
+			(at 198.12 80.0099 0)
+			(effects
+				(font
+					(size 1.27 1.27)
+				)
+				(justify left)
+			)
+		)
+		(property "Value" "IRLML6344"
+			(at 198.12 82.5499 0)
+			(effects
+				(font
+					(size 1.27 1.27)
+				)
+				(justify left)
+			)
+		)
+		(property "Footprint" "IRLML6344TRPBF:SOT95P240X112-3N"
+			(at 191.77 81.28 0)
 			(effects
 				(font
@@
 		)
 		(property "Datasheet" ""
-			(at 200.66 81.28 0)
+			(at 191.77 81.28 0)
 			(effects
 				(font
@@
 		)
 		(property "Description" ""
-			(at 200.66 81.28 0)
+			(at 191.77 81.28 0)
 			(effects
 				(font
@@
 		)
 		(property "MF" "Infineon Technologies"
-			(at 200.66 81.28 0)
+			(at 191.77 81.28 0)
 			(effects
 				(font
@@
 		)
 		(property "MAXIMUM_PACKAGE_HEIGHT" "19.3mm"
-			(at 200.66 81.28 0)
+			(at 191.77 81.28 0)
 			(effects
 				(font
@@
 		)
 		(property "Package" "TO-220 Infineon"
-			(at 200.66 81.28 0)
+			(at 191.77 81.28 0)
 			(effects
 				(font
@@
 		)
 		(property "Price" "None"
-			(at 200.66 81.28 0)
+			(at 191.77 81.28 0)
 			(effects
 				(font
@@
 		)
 		(property "Check_prices" "https://www.snapeda.com/parts/IRLZ44N/Infineon/view-part/?ref=eda"
-			(at 200.66 81.28 0)
+			(at 191.77 81.28 0)
 			(effects
 				(font
@@
 		)
 		(property "STANDARD" "IPC-7351B"
-			(at 200.66 81.28 0)
+			(at 191.77 81.28 0)
 			(effects
 				(font
@@
 		)
 		(property "PARTREV" "11/11/03"
-			(at 200.66 81.28 0)
+			(at 191.77 81.28 0)
 			(effects
 				(font
@@
 		)
 		(property "SnapEDA_Link" "https://www.snapeda.com/parts/IRLZ44N/Infineon/view-part/?ref=snap"
-			(at 200.66 81.28 0)
+			(at 191.77 81.28 0)
 			(effects
 				(font
@@
 		)
 		(property "MP" "IRLZ44N"
-			(at 200.66 81.28 0)
+			(at 191.77 81.28 0)
 			(effects
 				(font
@@
 		)
 		(property "Description_1" "N-Channel 55 V 47A (Tc) 3.8W (Ta), 110W (Tc) Surface Mount D2PAK"
-			(at 200.66 81.28 0)
+			(at 191.77 81.28 0)
 			(effects
 				(font
@@
 		)
 		(property "Availability" "In Stock"
-			(at 200.66 81.28 0)
+			(at 191.77 81.28 0)
 			(effects
 				(font
@@
 		)
 		(property "MANUFACTURER" "Infineon"
-			(at 200.66 81.28 0)
+			(at 191.77 81.28 0)
 			(effects
 				(font
@@
 			)
 		)
-		(property "Footprint" "Connector_AMASS:AMASS_XT30PW-M_1x02_P2.50mm_Horizontal"
+		(property "Footprint" "Connector_JST:JST_GH_SM02B-GHS-TB_1x02-1MP_P1.25mm_Horizontal"
 			(at 231.14 80.01 0)
 			(effects
@@
 			)
 		)
-		(property "Footprint" "Connector_AMASS:AMASS_XT30PW-M_1x02_P2.50mm_Horizontal"
+		(property "Footprint" "Connector_JST:JST_GH_SM02B-GHS-TB_1x02-1MP_P1.25mm_Horizontal"
 			(at 236.22 39.37 0)
 			(effects
